File: Project/matrix.kicad_sch (KiCad schematic)
At the start: 49 parts, among them SW1 RotaryEncoder_Switch

Commit message: firmware
Connections:
- net ROW3 renamed ROW2
Changed lines of the file:
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@@
 		)
 	)
-	(global_label "ROW3"
+	(global_label "ROW2"
 		(shape input)
 		(at 25.4 80.01 180)
